Commit message: Enable diff_drive module in default robot

File: assets/default/robots/diff_drive/robot.urdf (robot description, URDF)
Before this commit: robot sam_bot, 6 links, 5 joints
Links:
- removed link caster_rod2_left
Joints:
- removed joint caster_joint2
- joint caster_joint: child caster_rod2_left -> front_caster

Commit message: Organize default urdf

File: assets/default/robots/diff_drive/robot.urdf (robot description, URDF)
Before this commit: robot sam_bot, 5 links, 4 joints
Links:
- removed link base_footprint
- removed link base_link
- removed link caster_rod_left
- removed link front_caster
- removed link imu_link
Joints:
- removed joint base_joint
- removed joint caster_joint
- removed joint caster_rod_joint
- removed joint imu_joint
