Commit message: Improve heading stability of default robot

File: assets/default/robots/diff_drive/wheel_front.urdf (robot description, URDF)
Before this commit: robot None, 2 links, 2 joints
Links:
- added link caster_rod2_left; visual box size=0.02 0.02 0.1
Joints:
- added joint caster_joint2: type continuous, parent caster_rod2_left, child front_caster, origin xyz=0.0 0.0 0.0 rpy=0 0 0, axis 1.0 0.0 0.0
- joint caster_joint: child front_caster -> caster_rod2_left
